Commit message: Develop working environment

File: xarm_description/urdf/camera/realsense.gazebo.xacro (robot description, xacro)
@@ -23,5 +23,5 @@
         <update_rate>30</update_rate>
         <visualize>1</visualize>
-        <gz_frame_id>depth_frame</gz_frame_id>
+        <ignition_frame_id>world</ignition_frame_id>
         <topic>camera/depth</topic>
       </sensor>
@@ -49,5 +49,5 @@
         <update_rate>30</update_rate>
         <visualize>1</visualize>
-        <gz_frame_id>rbg_frame</gz_frame_id>
+        <gz_frame_id>world</gz_frame_id>
         <topic>camera/rgb</topic>
       </sensor>
@@ -75,5 +75,5 @@
         <update_rate>30</update_rate>
         <visualize>0</visualize>
-        <gz_frame_id>ir_frame</gz_frame_id>
+        <gz_frame_id>world</gz_frame_id>
         <topic>camera/ir1</topic>
       </sensor>
@@ -101,5 +101,5 @@
         <update_rate>30</update_rate>
         <visualize>0</visualize>
-        <gz_frame_id>ir_frame</gz_frame_id>
+        <gz_frame_id>world</gz_frame_id>
         <topic>camera/ir2</topic>
       </sensor>

File: xarm_description/urdf/common/common.gazebo.xacro (robot description, xacro)
@@ -1,4 +1,12 @@
 <?xml version="1.0"?>
 <robot xmlns:xacro="http://ros.org/wiki/xacro">
+  <xacro:macro name="gz_ros2_control_plugin" params="prefix:='' ros2_control_params:=''">
+    <gazebo>
+      <!-- Joint state publisher -->
+      <plugin filename="libgz_ros2_control-system.so" name="gz_ros2_control::GazeboSimROS2ControlPlugin">
+        <parameters>${ros2_control_params}</parameters>
+      </plugin>
+    </gazebo>
+  </xacro:macro>
   <xacro:macro name="ignition_ros2_control_plugin" params="prefix:='' ros2_control_params:=''">
     <gazebo>

File: xarm_description/urdf/xarm_device.urdf.xacro (robot description, xacro)
@@ -17,5 +17,5 @@
   <xacro:arg name="ros2_control_plugin" default="uf_robot_hardware/UFRobotSystemHardware"/>
   <xacro:arg name="ros2_control_params" default=""/>
-  <xacro:arg name="add_realsense_d435i" default="false"/>
+  <xacro:arg name="add_realsense_d435i" default="true"/>
   <xacro:arg name="add_d435i_links" default="true"/>
   <xacro:arg name="use_gazebo_camera" default="false"/>

File: xarm_description/urdf/xarm_device_macro.xacro (robot description, xacro)
@@ -52,9 +52,9 @@
     <!-- Specify Mesh file path -->
     <xacro:property name="mesh_suffix" value="${mesh_suffix}" scope="parent"/>
-    <xacro:if value="${ros2_control_plugin == 'gazebo_ros2_control/GazeboSystem' or ros2_control_plugin == 'ign_ros2_control/IgnitionSystem'}">
+    <xacro:if value="${ros2_control_plugin == 'gazebo_ros2_control/GazeboSystem' or ros2_control_plugin == 'ign_ros2_control/IgnitionSystem' or ros2_control_plugin == 'gz_ros2_control/GazeboSimSystem'}">
       <!-- gazebo use -->
       <xacro:property name="mesh_path" value="file://$(find xarm_description)/meshes" scope="parent"/>
     </xacro:if>
-    <xacro:unless value="${ros2_control_plugin == 'gazebo_ros2_control/GazeboSystem' or ros2_control_plugin == 'ign_ros2_control/IgnitionSystem'}">
+    <xacro:unless value="${ros2_control_plugin == 'gazebo_ros2_control/GazeboSystem' or ros2_control_plugin == 'ign_ros2_control/IgnitionSystem' or ros2_control_plugin == 'gz_ros2_control/GazeboSimSystem'}">
       <xacro:property name="mesh_path" value="package://xarm_description/meshes" scope="parent"/>
     </xacro:unless>
@@ -200,4 +200,13 @@
       </xacro:unless>
     </xacro:unless>
+<!--    <xacro:if value="${add_realsense_d435i}">-->
+<!--      &lt;!&ndash; (xarm) Load RealSense D435i URDF &ndash;&gt;-->
+<!--      <xacro:include filename="$(find xarm_description)/urdf/camera/realsense_d435i.urdf.xacro" />-->
+<!--      <xacro:d435i_urdf prefix="${prefix}" add_d435i_links="${add_d435i_links}" />-->
+<!--      <xacro:if value="${add_d435i_links}">-->
+<!--        <xacro:include filename="$(find xarm_description)/urdf/camera/realsense.gazebo.xacro" />    -->
+<!--        <xacro:realsense_gazebo prefix="${prefix}" />-->
+<!--      </xacro:if>-->
+<!--    </xacro:if>-->
     <xacro:if value="${add_realsense_d435i}">
       <!-- (xarm) Load RealSense D435i URDF -->
@@ -278,6 +287,9 @@
           <xacro:ignition_ros2_control_plugin prefix="${prefix}" ros2_control_params="${new_ros2_control_params}"/>
         </xacro:if>
+<!--        <xacro:unless value="${ros2_control_plugin == 'ign_ros2_control/IgnitionSystem'}">-->
+<!--          <xacro:gazebo_ros2_control_plugin ros2_control_params="${new_ros2_control_params}"/>-->
+<!--        </xacro:unless>-->
         <xacro:unless value="${ros2_control_plugin == 'ign_ros2_control/IgnitionSystem'}">
-          <xacro:gazebo_ros2_control_plugin ros2_control_params="${new_ros2_control_params}"/>
+          <xacro:gz_ros2_control_plugin ros2_control_params="${new_ros2_control_params}"/>
         </xacro:unless>
       </xacro:if>

Commit message: Add second camera sensor

File: xarm_description/urdf/camera/realsense.gazebo.xacro (robot description, xacro)
@@ -3,5 +3,5 @@
   <xacro:macro name="realsense_gazebo" params="prefix:='' ">
     <gazebo reference="${prefix}camera_depth_frame">
-      <sensor name="cameradepth" type="depth">
+      <sensor name="${prefix}cameradepth" type="depth">
         <camera name="camera">
           <horizontal_fov>1.57</horizontal_fov>
@@ -23,10 +23,10 @@
         <update_rate>30</update_rate>
         <visualize>1</visualize>
+        <gz_frame_id>world</gz_frame_id>
         <ignition_frame_id>world</ignition_frame_id>
-        <topic>camera/depth</topic>
       </sensor>
     </gazebo>
     <gazebo reference="${prefix}camera_color_frame">
-      <sensor name="cameracolor" type="camera">
+      <sensor name="${prefix}cameracolor" type="camera">
         <camera name="camera">
           <horizontal_fov>1.57</horizontal_fov>
@@ -50,9 +50,8 @@
         <visualize>1</visualize>
         <gz_frame_id>world</gz_frame_id>
-        <topic>camera/rgb</topic>
       </sensor>
     </gazebo>
     <gazebo reference="${prefix}camera_left_ir_frame">
-      <sensor name="cameraired1" type="camera">
+      <sensor name="${prefix}cameraired1" type="camera">
         <camera name="camera">
           <horizontal_fov>1.57</horizontal_fov>
@@ -74,11 +73,10 @@
         <always_on>1</always_on>
         <update_rate>30</update_rate>
-        <visualize>0</visualize>
+        <visualize>1</visualize>
         <gz_frame_id>world</gz_frame_id>
-        <topic>camera/ir1</topic>
       </sensor>
     </gazebo>
     <gazebo reference="${prefix}camera_right_ir_frame">
-      <sensor name="cameraired2" type="camera">
+      <sensor name="${prefix}cameraired2" type="camera">
         <camera name="camera">
           <horizontal_fov>1.57</horizontal_fov>
@@ -100,15 +98,7 @@
         <always_on>1</always_on>
         <update_rate>30</update_rate>
-        <visualize>0</visualize>
+        <visualize>1</visualize>
         <gz_frame_id>world</gz_frame_id>
-        <topic>camera/ir2</topic>
       </sensor>
-    </gazebo>
-    <gazebo>
-      <plugin
-        filename="gz-sim-sensors-system"
-        name="gz::sim::systems::Sensors">
-      <render_engine>ogre2</render_engine>
-      </plugin>
     </gazebo>
     <!-- <gazebo>

File: xarm_description/urdf/camera/realsense_d435i.urdf.xacro (robot description, xacro)
@@ -9,5 +9,5 @@
         origin_xyz="0 0 0"
         origin_rpy="0 0 0"
-        material_name="${prefix}Silver" />
+        material_name="Silver" />
       <xacro:common_link_collision
         mesh_filename="camera/realsense/collision/d435_with_cam_stand"

File: xarm_description/urdf/xarm_device.urdf.xacro (robot description, xacro)
@@ -19,4 +19,5 @@
   <xacro:arg name="add_realsense_d435i" default="true"/>
   <xacro:arg name="add_d435i_links" default="true"/>
+  <xacro:arg name="add_dual_realsense" default="true"/>
   <xacro:arg name="use_gazebo_camera" default="false"/>
   <xacro:arg name="add_other_geometry" default="false"/>
@@ -48,4 +49,5 @@
     load_gazebo_plugin="true" ros2_control_params="$(arg ros2_control_params)"
     add_realsense_d435i="$(arg add_realsense_d435i)"
+    add_dual_realsense="$(arg add_dual_realsense)"
     add_d435i_links="$(arg add_d435i_links)"
     add_other_geometry="$(arg add_other_geometry)"

File: xarm_description/urdf/xarm_device_macro.xacro (robot description, xacro)
@@ -21,4 +21,5 @@
     add_realsense_d435i:=false
     add_d435i_links:=true
+    add_dual_realsense:=false
     use_gazebo_camera:=false
     add_other_geometry:=false
@@ -200,21 +201,43 @@
       </xacro:unless>
     </xacro:unless>
-<!--    <xacro:if value="${add_realsense_d435i}">-->
-<!--      &lt;!&ndash; (xarm) Load RealSense D435i URDF &ndash;&gt;-->
-<!--      <xacro:include filename="$(find xarm_description)/urdf/camera/realsense_d435i.urdf.xacro" />-->
-<!--      <xacro:d435i_urdf prefix="${prefix}" add_d435i_links="${add_d435i_links}" />-->
-<!--      <xacro:if value="${add_d435i_links}">-->
-<!--        <xacro:include filename="$(find xarm_description)/urdf/camera/realsense.gazebo.xacro" />    -->
-<!--        <xacro:realsense_gazebo prefix="${prefix}" />-->
-<!--      </xacro:if>-->
-<!--    </xacro:if>-->
     <xacro:if value="${add_realsense_d435i}">
+      <gazebo>
+        <plugin
+          filename="gz-sim-sensors-system"
+          name="gz::sim::systems::Sensors">
+          <render_engine>ogre2</render_engine>
+        </plugin>
+      </gazebo>
       <!-- (xarm) Load RealSense D435i URDF -->
       <xacro:include filename="$(find xarm_description)/urdf/camera/realsense_d435i.urdf.xacro" />
-      <xacro:d435i_urdf prefix="${prefix}" add_d435i_links="${add_d435i_links}" />
-      <xacro:if value="${add_d435i_links}">
-        <xacro:include filename="$(find xarm_description)/urdf/camera/realsense.gazebo.xacro" />
-        <xacro:realsense_gazebo prefix="${prefix}" />
-      </xacro:if>
+      <!-- add two sensors -->
+      <xacro:if value="${add_dual_realsense}">
+        <!--  Add Left Camera-->
+        <xacro:d435i_urdf prefix="${prefix}left_" add_d435i_links="${add_d435i_links}"/>
+        <xacro:d435i_urdf prefix="${prefix}right_" add_d435i_links="${add_d435i_links}"/>
+        <xacro:if value="${add_d435i_links}">
+          <xacro:include filename="$(find xarm_description)/urdf/camera/realsense.gazebo.xacro" />
+          <xacro:realsense_gazebo prefix="${prefix}left_" />
+          <xacro:realsense_gazebo prefix="${prefix}right_" />
+          <link name="${prefix}link_eef"/>
+          <joint name="${prefix}eef_left_camera" type="fixed">
+          <origin xyz="0 0 0" rpy="0 0 -1.2" />
+          <parent link="${prefix}link_eef" />
+          <child link="${prefix}left_link_eef" />
+          </joint>
+          <joint name="${prefix}eef_right_camera" type="fixed">
+          <origin xyz="0 0 0.004" rpy="0 0 1.2" />
+          <parent link="${prefix}link_eef" />
+          <child link="${prefix}right_link_eef" />
+          </joint>
+        </xacro:if>
+      </xacro:if>
+      <xacro:unless value="${add_dual_realsense}">
+        <xacro:d435i_urdf prefix="${prefix}" add_d435i_links="${add_d435i_links}" />
+        <xacro:if value="${add_d435i_links}">
+          <xacro:include filename="$(find xarm_description)/urdf/camera/realsense.gazebo.xacro" />
+          <xacro:realsense_gazebo prefix="${prefix}" />
+        </xacro:if>
+      </xacro:unless>
     </xacro:if>
     <xacro:unless value="${add_realsense_d435i}">

Commit message: Debug plugin failure

File: xarm_description/urdf/camera/realsense.gazebo.xacro (robot description, xacro)
@@ -12,5 +12,5 @@
           <clip>
             <near>0.1</near>
-            <far>100</far>
+            <far>1</far>
           </clip>
           <noise>
@@ -37,5 +37,5 @@
           <clip>
             <near>0.1</near>
-            <far>100</far>
+            <far>1</far>
           </clip>
           <noise>
@@ -62,5 +62,5 @@
           <clip>
             <near>0.1</near>
-            <far>100</far>
+            <far>1</far>
           </clip>
           <noise>
@@ -87,5 +87,5 @@
           <clip>
             <near>0.1</near>
-            <far>100</far>
+            <far>1</far>
           </clip>
           <noise>
@@ -101,5 +101,5 @@
       </sensor>
     </gazebo>
-    <!-- <gazebo>
+    <gazebo>
       <plugin name="realsense_gazebo_camera" filename="librealsense_gazebo_plugin.so">
         <prefix>camera</prefix>
@@ -125,5 +125,5 @@
         <pointCloudCutoff>0.3</pointCloudCutoff>
       </plugin>
-    </gazebo> -->
+    </gazebo>
   </xacro:macro>
 </robot>

File: xarm_description/urdf/camera/realsense_d435i.urdf.xacro (robot description, xacro)
@@ -10,8 +10,8 @@
         origin_rpy="0 0 0"
         material_name="Silver" />
-      <xacro:common_link_collision
-        mesh_filename="camera/realsense/collision/d435_with_cam_stand"
-        origin_xyz="0 0 0"
-        origin_rpy="0 0 0" />
+<!--      <xacro:common_link_collision -->
+<!--        mesh_filename="camera/realsense/collision/d435_with_cam_stand"  -->
+<!--        origin_xyz="0 0 0" -->
+<!--        origin_rpy="0 0 0" />-->
     </link>
     <xacro:if value="${add_d435i_links}">

File: xarm_description/urdf/xarm_device_macro.xacro (robot description, xacro)
@@ -221,13 +221,20 @@
           <xacro:realsense_gazebo prefix="${prefix}right_" />
           <link name="${prefix}link_eef"/>
-          <joint name="${prefix}eef_left_camera" type="fixed">
-          <origin xyz="0 0 0" rpy="0 0 -1.2" />
-          <parent link="${prefix}link_eef" />
+          <joint name="${prefix}arm_left_camera" type="fixed">
+          <origin xyz="0 0 00.0035" rpy="0 0 -1.2" />
+<!--          <parent link="${prefix}link_eef" />-->
+          <parent link="${prefix}link${dof}" />
           <child link="${prefix}left_link_eef" />
           </joint>
-          <joint name="${prefix}eef_right_camera" type="fixed">
-          <origin xyz="0 0 0.004" rpy="0 0 1.2" />
-          <parent link="${prefix}link_eef" />
+          <joint name="${prefix}left_right_camera" type="fixed">
+          <origin xyz="0 0 0.0035" rpy="0 0 2.4" />
+<!--          <parent link="${prefix}link_eef" />-->
+          <parent link="${prefix}left_link_eef" />
           <child link="${prefix}right_link_eef" />
+          </joint>
+          <joint name="${prefix}right_camera_eef" type="fixed">
+          <origin xyz="0 0 0.0035" rpy="0 0 -1.20" />
+          <parent link="${prefix}right_link_eef" />
+          <child link="${prefix}link_eef" />
           </joint>
         </xacro:if>
@@ -241,12 +248,20 @@
       </xacro:unless>
     </xacro:if>
-    <xacro:unless value="${add_realsense_d435i}">
+<!--    <xacro:unless value="${add_realsense_d435i}">-->
+<!--      <link name="${prefix}link_eef"/>-->
+<!--    </xacro:unless>-->
+<!--    <joint name="${prefix}joint_eef" type="fixed">-->
+<!--      <origin xyz="0 0 0" rpy="0 0 0" />-->
+<!--      <parent link="${prefix}link${dof}" />-->
+<!--      <child link="${prefix}link_eef" />-->
+<!--    </joint>    -->
+  <xacro:unless value="${add_realsense_d435i}">
       <link name="${prefix}link_eef"/>
-    </xacro:unless>
-    <joint name="${prefix}joint_eef" type="fixed">
-      <origin xyz="0 0 0" rpy="0 0 0" />
-      <parent link="${prefix}link${dof}" />
-      <child link="${prefix}link_eef" />
-    </joint>
+      <joint name="${prefix}joint_eef" type="fixed">
+        <origin xyz="0 0 0" rpy="0 0 0" />
+        <parent link="${prefix}link${dof}" />
+        <child link="${prefix}link_eef" />
+      </joint>
+  </xacro:unless>
     <xacro:if value="${add_gripper}">
       <xacro:if value="${robot_type == 'lite'}">
